File: Audio.kicad_sch (KiCad schematic)
At the start: 28 parts, among them J3 AUDIO JACK, J4 MEM2061-01-188-00-A, J5 1x6 header, Q4 BC846, U6 PCM5102

Commit message: Updated schematics/ pcb
Parts:
- renumbered BCK to BCK1, DOUT to DOUT1, LRCK to LRCK1, OUTL to OUTL1, OUTR to OUTR1
Changed lines of the file:
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@@
 		(on_board yes)
 		(dnp no)
-		(property "Reference" "LRCK"
+		(property "Reference" "LRCK1"
 			(at 25.654 26.416 0)
 			(effects
@@
 			(project "Radiation"
 				(path "/0a781558-ebe5-4562-8748-3cbe471da24e/b03a8cbd-5823-419c-808a-8b6445fe34d3"
-					(reference "LRCK")
+					(reference "LRCK1")
 					(unit 1)
 				)
@@
 		(on_board yes)
 		(dnp no)
-		(property "Reference" "OUTL"
+		(property "Reference" "OUTL1"
 			(at 76.962 84.836 0)
 			(effects
@@
 			(project "Radiation"
 				(path "/0a781558-ebe5-4562-8748-3cbe471da24e/b03a8cbd-5823-419c-808a-8b6445fe34d3"
-					(reference "OUTL")
+					(reference "OUTL1")
 					(unit 1)
 				)
@@
 		(on_board yes)
 		(dnp no)
-		(property "Reference" "OUTR"
+		(property "Reference" "OUTR1"
 			(at 73.152 82.296 0)
 			(effects
@@
 			(project "Radiation"
 				(path "/0a781558-ebe5-4562-8748-3cbe471da24e/b03a8cbd-5823-419c-808a-8b6445fe34d3"
-					(reference "OUTR")
+					(reference "OUTR1")
 					(unit 1)
 				)
@@
 		(on_board yes)
 		(dnp no)
-		(property "Reference" "DOUT"
+		(property "Reference" "DOUT1"
 			(at 30.988 26.416 0)
 			(effects
@@
 			(project "Radiation"
 				(path "/0a781558-ebe5-4562-8748-3cbe471da24e/b03a8cbd-5823-419c-808a-8b6445fe34d3"
-					(reference "DOUT")
+					(reference "DOUT1")
 					(unit 1)
 				)
@@
 		(on_board yes)
 		(dnp no)
-		(property "Reference" "BCK"
+		(property "Reference" "BCK1"
 			(at 36.83 26.416 0)
 			(effects
@@
 			(project "Radiation"
 				(path "/0a781558-ebe5-4562-8748-3cbe471da24e/b03a8cbd-5823-419c-808a-8b6445fe34d3"
-					(reference "BCK")
+					(reference "BCK1")
 					(unit 1)
 				)

Commit message: revisions after design review by Ted Yapo
Parts:
- removed R25, R26, R27: 33R, Resistor_SMD:R_0805_2012Metric, symbol Device:R_US
- added C26: 2.2uF, Capacitor_SMD:C_0805_2012Metric, symbol Device:C
Connections:
- net AGND: now also J3.1, U6.12 (SCK), U6.19 (DGND), C26.2; no longer J3.3, U6.5 (VNEG)
- net I2S_BCK: now also U6.13 (BCK)
- net I2S_DOUT: now also U6.14 (DIN)
- net I2S_LRCK: now also U6.15 (LRCK)
- net OUTR: now also J3.3; no longer J3.1
- net at C16.1, C17.1, U6.18 (LDOO): no longer U6.19 (DGND)
- new net: C26.1, U6.5 (VNEG)
- no-connect marks 5 -> 4
Other:
- moved on the sheet: C14, C15, C18, C19, J3, OUTL1, OUTR1, R29, U6
