File: Power.kicad_sch (KiCad schematic)
At the start: 52 parts, among them Q1 AO3400A, T1 FL2810-1L, U1 TPS2115APWR, U2 RP115X, U3 TPS613222ADBV

Commit message: proto 1 final
Parts:
- U1: footprint PW8 -> TPS2115APWR:PW8
Changed lines of the file:
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@@
 			)
 		)
-		(property "Footprint" "PW8"
+		(property "Footprint" "TPS2115APWR:PW8"
 			(at 45.72 41.91 0)
 			(effects
