File: _autosave-Audio.kicad_sch (KiCad schematic)
At the start: 26 parts, among them J3 AUDIO JACK, J4 MEM2061-01-188-00-A, J5 1x6 header, Q4 BC846, U6 PCM5102

Commit message: proto 1 final
Parts:
- J4: footprint MEM2061-01-188-00-A_GCT -> MEM2061 SD CARD CONNECTOR:MEM2061-01-188-00-A_GCT
Changed lines of the file:
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@@
 			)
 		)
-		(property "Footprint" "MEM2061-01-188-00-A_GCT"
+		(property "Footprint" "MEM2061 SD CARD CONNECTOR:MEM2061-01-188-00-A_GCT"
 			(at 125.73 167.64 0)
 			(effects
