File: Audio2.kicad_sch (KiCad schematic)
At the start: 26 parts, among them J3 AUDIO JACK, J4 MEM2061-01-188-00-A, J5 1x6 header, Q4 BC846, U6 PCM5102

Commit message: updates
Other:
- note added: "RADIATION INPUT TO MCU"
- moved on the sheet: S4

Commit message: updates
Other:
- note removed: "RADIATION INPUT TO MCU"

Commit message: PCB v2
Connections:
- net GPIO15 is gone; now on net GPIO16: S4.5B
- net +3.3V: no longer S4.6A
- net GPIO16: no longer S4.6B
- new net RAD_IN: S4.6A
- new net RAD_IN2: S4.6B
Changed lines of the file:
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@@
-	)
-	(junction
-		(at 196.85 156.21)
-		(diameter 0)
-		(color 0 0 0 0)
 	)
 	(junction
@@
 	(wire
 		(pts
-			(xy 212.09 161.29) (xy 196.85 161.29)
-		)
-		(stroke
-			(width 0)
-			(type default)
-		)
-	)
-	(wire
-		(pts
 			(xy 196.85 156.21) (xy 212.09 156.21)
 		)
@@
 	(wire
 		(pts
+			(xy 227.33 161.29) (xy 247.65 161.29)
+		)
+		(stroke
+			(width 0)
+			(type default)
+		)
+	)
+	(wire
+		(pts
 			(xy 29.21 173.99) (xy 43.18 173.99)
 		)
@@
 	(wire
 		(pts
-			(xy 227.33 161.29) (xy 247.65 161.29)
-		)
-		(stroke
-			(width 0)
-			(type default)
-		)
-	)
-	(wire
-		(pts
 			(xy 106.68 64.77) (xy 115.57 64.77)
 		)
@@
 		)
 	)
-	(polyline
-		(pts
-			(xy 176.53 163.83) (xy 280.67 163.83)
-		)
-		(stroke
-			(width 0)
-			(type default)
-		)
-	)
 	(wire
 		(pts
@@
 	(wire
 		(pts
+			(xy 196.85 161.29) (xy 212.09 161.29)
+		)
+		(stroke
+			(width 0)
+			(type default)
+		)
+	)
+	(wire
+		(pts
 			(xy 106.68 59.69) (xy 115.57 59.69)
 		)
@@
 		(pts
 			(xy 31.75 43.18) (xy 29.21 43.18)
-		)
-		(stroke
-			(width 0)
-			(type default)
-		)
-	)
-	(wire
-		(pts
-			(xy 196.85 156.21) (xy 196.85 161.29)
 		)
 		(stroke
@@
 		)
 	)
+	(label "RAD_IN2"
+		(at 232.41 161.29 0)
+		(fields_autoplaced yes)
+		(effects
+			(font
+				(size 1.27 1.27)
+			)
+			(justify left bottom)
+		)
+	)
 	(label "MUTE"
 		(at 55.88 50.8 0)
@@
 	(label "I2S_LRCK"
 		(at 39.37 46.99 0)
+		(fields_autoplaced yes)
+		(effects
+			(font
+				(size 1.27 1.27)
+			)
+			(justify left bottom)
+		)
+	)
+	(label "RAD_IN"
+		(at 200.66 161.29 0)
 		(fields_autoplaced yes)
 		(effects
@@
 		)
 	)
+	(hierarchical_label "RAD_IN"
+		(shape input)
+		(at 196.85 161.29 180)
+		(fields_autoplaced yes)
+		(effects
+			(font
+				(size 1.27 1.27)
+			)
+			(justify right)
+		)
+	)
 	(hierarchical_label "MUTE"
 		(shape input)
@@
 		)
 	)
+	(hierarchical_label "RAD_IN2"
+		(shape input)
+		(at 247.65 161.29 0)
+		(fields_autoplaced yes)
+		(effects
+			(font
+				(size 1.27 1.27)
+			)
+			(justify left)
+		)
+	)
 	(hierarchical_label "SCK"
 		(shape input)
@@
 		)
 	)
-	(hierarchical_label "GPIO15"
+	(hierarchical_label "GPIO16"
 		(shape input)
 		(at 247.65 156.21 0)
@@
 		(fields_autoplaced yes)
 		(effects
-			(font
-				(size 1.27 1.27)
-			)
-			(justify left)
-		)
-	)
-	(hierarchical_label "GPIO16"
-		(shape input)
-		(at 247.65 161.29 0)
-		(fields_autoplaced yes)
-		(effects
