File: MCU2.kicad_sch (KiCad schematic)
At the start: 37 parts, among them J1 USB4105-GF-A, J2 USB4105-GF-A, Q2 2N7002-TP, Q3 2N7002-TP, U4 ESP32-S3-WROOM-1-N8, U5 FT231XS

Commit message: updates
Parts:
- added GND1: TestPoint, Connector_Pin:Pin_D1.0mm_L10.0mm, symbol Connector:TestPoint
- Q2, Q3: footprint Package_TO_SOT_THT:TO-92_Inline -> Package_TO_SOT_SMD:SOT-23
Connections:
- net GND: now also GND1.1

Commit message: updates
Connections:
- net BLINK: now reaches U4.38 (IO2)
- no-connect marks 20 -> 19
Changed lines of the file:
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@@
-	)
-	(no_connect
-		(at 217.17 66.04)
 	)
 	(no_connect
@@
 		(pts
 			(xy 26.67 146.05) (xy 26.67 147.32)
+		)
+		(stroke
+			(width 0)
+			(type default)
+		)
+	)
+	(wire
+		(pts
+			(xy 217.17 66.04) (xy 226.06 66.04)
 		)
 		(stroke
@@
 		)
 	)
+	(label "BLINK"
+		(at 218.44 66.04 0)
+		(fields_autoplaced yes)
+		(effects
+			(font
+				(size 1.27 1.27)
+			)
+			(justify left bottom)
+		)
+	)
 	(label "GPIO46"
 		(at 162.56 40.64 0)
@@
 		)
 	)
+	(hierarchical_label "BLINK"
+		(shape input)
+		(at 226.06 66.04 0)
+		(fields_autoplaced yes)
+		(effects
+			(font
+				(size 1.27 1.27)
+			)
+			(justify left)
+		)
+	)

Commit message: PCB v2
Parts:
- removed D10, D11, D12, D5, D6, D7: ESD9B5.0ST5G, Diode_SMD:D_SOD-923, symbol Diode:ESD9B5.0ST5G
- added D10, D11, D12, D5, D6, D7: PESD5V0S1BA, SOD323_NXP, symbol PESD5V0S1BA:PESD5V0S1BA
- added GND2: TestPoint, Connector_Pin:Pin_D1.0mm_L10.0mm, symbol Connector:TestPoint
Connections:
- net +VBAT is gone; now on net VBUS: R9.2
- net DP_N: now also D11.2
- net DP_P: now also D12.2
- net GND: now also D10.1, D11.1, D12.1, D5.1, D6.1, D7.1, GND2.1
- net USB_D+: now also D5.2
- net USB_D-: now also D6.2
- net VBUS: now also D10.2, D7.2
- net BAT_SENSE: now reaches U4.17 (IO9)
- net GPIO15 renamed RAD_IN2
- net VSTAT: no longer names the net of U4.15 (IO3)
- no-connect marks 19 -> 20
Other:
- moved on the sheet: C11, C12, C25, R14, R15, R21, R31, U5
