File: Power2.kicad_sch (KiCad schematic)
At the start: 57 parts, among them Q1 AO3400A, T1 FL2810-1L, U2 RP115X, U3 TPS613222ADBV

Commit message: updates
Parts:
- removed 3.3V1, VBUS: TestPoint, Connector_Pin:Pin_D1.0mm_L10.0mm, symbol Connector:TestPoint
- removed C5, C6: 1uF, Capacitor_SMD:C_0805_2012Metric, symbol Device:C
- removed U2: RP115X, Package_TO_SOT_SMD:SOT-89-5, symbol Regulator_Linear:RP115X
- added C2, C3: 10uF, Capacitor_SMD:C_0805_2012Metric, symbol Device:C
- added D16: YELLOW, LED_SMD:LED_0805_2012Metric, symbol Device:LED
- added R36: 4.7k, Resistor_SMD:R_0805_2012Metric, symbol Device:R_US
- added R4: 5M, Resistor_SMD:R_0805_2012Metric, symbol Device:R_US
- added U1: AP7363-33D-13, TO252-3L_DIO, symbol AP7363_33D_13:AP7363-33D-13
- C27: value 220uF/ 500V -> 150uF/ 450V; footprint Capacitor_SMD:C_2220_5750Metric -> Capacitor_THT:CP_Radial_D18.0mm_P7.50mm; MPN ECW-FD2J105K -> UCP2W151MHD
- D4: value GREEN -> YELLOW; MPN 150080GS75000 -> 150080YS75000
- renumbered CX to CX1, CX to CX2, RX to RX1, UX to UX1
Connections:
- net +3.3V: now also L1.1, C3.1, R4.2, U1.3 (OUT)
- net +5V: now also R36.2; no longer R8.2
- net GND: now also C2.2, C3.2, D16.1 (K), U1.2 (GND)
- net VBUS: now also C2.1, U1.1 (IN)
- net VHIGH: no longer L1.1
- new net: D16.2 (A), R36.1
- new net BLINK: R8.2
Other:
- note added: "Delon Voltage Doubler Circuit"
- note removed: "1. Breadboard Delon circuit with input to MCU 2. set PCB up for both with jumpers! 3. design and test input to the ESP32 4. add all of these things to PCB and BOM 5. test SD card and audio footprint 6. change 3.3V regulator part 7. check BOM to make sure everything is on it 8. 40 pushups! did 30"
- moved on the sheet: 5V1, C4, C7, C8, D13, D14, D2, D3, HIV-1, L1, R23, R24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

Commit message: PCB v2
Parts:
- removed C27: 150uF/ 450V, Capacitor_THT:CP_Radial_D18.0mm_P7.50mm, symbol Device:C
- removed STAT1: TestPoint, Connector_Pin:Pin_D1.0mm_L10.0mm, symbol Connector:TestPoint
- added C30, C5: 1000pF, Capacitor_SMD:C_0805_2012Metric, symbol Device:C
- added C6: 0.1uF, Capacitor_SMD:C_0805_2012Metric, symbol Device:C
- added JP4, JP5, JP6: SolderJumper_2_Open, Jumper:SolderJumper-2_P1.3mm_Open_RoundedPad1.0x1.5mm, symbol Jumper:SolderJumper_2_Open
- added R37: 100R, Resistor_SMD:R_0805_2012Metric, symbol Device:R_US
- added R38: 1M, Resistor_SMD:R_1210_3225Metric, symbol Device:R_US
- added R39: 22k, Resistor_SMD:R_0805_2012Metric, symbol Device:R_US
- added R40, R41: 10k, Resistor_SMD:R_0805_2012Metric, symbol Device:R_US
- added U2: LM393BIPWR, LM393BIPWR:PW0008A-MFG, symbol LM393BIPWR:LM393BIPWR
- C28: value 0.01uF -> 100pF; ALT MPN (none) -> C0805C471K5RACTU; MPN C0805C103K5RACTU -> C0805C101J5GACTU
- R4: value 5M -> 10k; MPN (none) -> CRCW08054K70FKEAC
- T1: Manufacturer_Name (none) -> Murata Electronics; Manufacturer_Part_Number (none) -> 54100C; Mouser Part Number (none) -> 580-54100C; Mouser Price/Stock (none) -> https://www.mouser.com/Search/Refine.aspx?Keyword=580-54100C
- U1: footprint TO252-3L_DIO -> AP7363_33D_13:TO252-3L_DIO
Connections:
- net +3.3V: now also C6.2, JP4.2 (B), R39.2, U2.8 (VCC)
- net GND: now also C28.2, C5.2, C6.1, JP5.2 (B), R37.1, R40.1, R41.1, U2.4 (GND); no longer C28.1
- net CATHODE: now reaches C29.1, D15.2 (A), F1.2, HIV-1.1
- net at DRAIN1.1, JP1.1 (A), JP2.1 (A)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: now also C5.1, R37.2; no longer C28.2
- net at PWM1.1, Q1.1 (G), R5.1: now also C28.1
- net ANODE: now reaches F1.1, R3.1
- net ANODE: now also C30.1
- net RAD_IN: now reaches R4.1
- net RAD_IN: now also U2.1 (1OUT)
- net +VBAT: no longer names the net of CX1.1, UX1.6 (IN2)
- net +VBAT: no longer R24.2
- net VHIGH: no longer names the net of UX1.7 (OUT)
- net VSTAT: no longer names the net of UX1.1 (STAT)
- new net: JP4.1 (A), U2.5 (2IN+)
- new net: JP5.1 (A), U2.6 (2IN-)
- new net: JP6.2 (B), U2.7 (2OUT)
- new net: R38.1, R41.2, U2.2 (1IN-)
- new net: C30.2, R38.2
- new net: R39.1, R40.2, U2.3 (1IN+)
- new net BAT_SENSE: R24.2
- no-connect marks 2 -> 3
Other:
- note added: "-"
- note added: "1V"
- note added: "IDLE at (-) 0V IDLE at (+) 1V IDLE OUTPUT 3.3V SWITCH PULSE at (-) -0V"
- note added: "IDLE: BETWN HIV+ AND HIV- = 420VDC IDLE: BETWN HIV+ AND R3/ ANODE = OPEN CIRCUIT SWITCH PULSE: BETWN HIV+ AND R3/ ANODE = NEGATIVE VOLTAGE"
- note added: "If the voltage at the inverting terminal (-) is greater than the voltage at the noninverting terminal (+), then the output of the op amp will be drawn down to ground, allowing electricity to flow from VCC to ground, turning on the output device. If the voltage at the inverting terminal (-) is less than at the noninverting terminal (+), then the output of the op amp stays at VCC allowing no electr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"
- note removed: "TESTED WITH 50kHz"
- moved on the sheet: C20, C22, C28, D14, D16, D2, PWM1, R24, R32, R33, R36, R4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

Commit message: update V2
Parts:
- JP1, JP2, JP4, JP5, JP6: now in the parts list
