File: Radiation2.kicad_pcb (KiCad board)
At the start: 4 copper layers, 102 x 125 mm, 115 parts, among them J1 USB4105-GF-A, J2 USB4105-GF-A, J3 AUDIO JACK, J4 MEM2061-01-188-00-A, J5 1x6 header, Q1 AO3400A, Q2 2N7002-TP, Q3 2N7002-TP, Q4 BC846, T1 FL2810-1L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

Commit message: updates
Parts:
- removed BCK, LRCK, TP3, TP5, TP8: TestPoint, Connector_Pin:Pin_D1.0mm_L10.0mm
- removed OUT L: TestPoint, Connector_Pin:Pin_D1.0mm_L10.0mm
- removed OUT R: TestPoint, Connector_Pin:Pin_D1.0mm_L10.0mm
- added BCK1: TestPoint, Connector_Pin:Pin_D1.0mm_L10.0mm, F.Cu at (136.0, 155.9)
- added C27: 1uF/ 500V, Capacitor_SMD:C_2220_5750Metric, F.Cu at (42.2, 56.4)
- added D15: ES1H, ES1H:DIOM4226X244N, F.Cu at (51.4, 56.0)
- added DRAIN1: TestPoint, Connector_Pin:Pin_D1.0mm_L10.0mm, F.Cu at (61.1, 67.7)
- added LRCK1: TestPoint, Connector_Pin:Pin_D1.0mm_L10.0mm, F.Cu at (134.7, 147.8)
- added OUTL1: TestPoint, Connector_Pin:Pin_D1.0mm_L10.0mm, F.Cu at (136.4, 179.1)
- added OUTR1: TestPoint, Connector_Pin:Pin_D1.0mm_L10.0mm, F.Cu at (136.4, 174.3)
- added R35: 10R, Resistor_SMD:R_2512_6332Metric, F.Cu at (61.3, 56.7)
- Q2, Q3: footprint Package_TO_SOT_THT:TO-92_Inline -> Package_TO_SOT_SMD:SOT-23
- R7: value 5R -> 10R
- moved F1 3.56 mm to (44.8, 184.9)
- moved Q2 1.33 mm to (71.1, 167.1)
- moved Q3 0.64 mm to (71.1, 162.5)
Connections:
- net /Audio/OUTL renamed /Audio2/OUTL
- net /Audio/OUTR renamed /Audio2/OUTR
- net /MCU/DP_N renamed /MCU2/DP_N
- net /MCU/DP_P renamed /MCU2/DP_P
- net /MCU/RX renamed /MCU2/RX
- net /MCU/RX_LED renamed /MCU2/RX_LED
- net /MCU/SHELL_GND renamed /MCU2/SHELL_GND
- net /MCU/TX renamed /MCU2/TX
- net /MCU/TX_LED renamed /MCU2/TX_LED
- D1 pad 2: +500V -> Net-(D1-A)
- PWM1 pad 1: /PWM -> Net-(Q1-G)
- T1 pad 2: +5V -> Net-(R35-Pad1)
Routing:
- net +500V: track 112.1 -> 80.4 mm
- net Net-(Q2-G): track 12.7 -> 0.00 mm
- net Net-(Q1-G): track 85.4 -> 76.9 mm
- net Net-(Q3-D): track 25.9 -> 19.7 mm
- net /GPIO0: track 166.0 -> 161.9 mm
- net GND: track 407.7 -> 403.9 mm
- net /EN: track 181.5 -> 177.9 mm
- net Net-(Q2-S): track 34.6 -> 37.6 mm
- net Net-(Q3-G): track 11.3 -> 9.87 mm
Other:
- board text added: "+"
- board text added: "-"
- board text added: "MESSAGES FROM SPACE PROTO 1.1 FEB 20, 2025"
- board text removed: "MESSAGES FROM SPACE PROTO 1.0 FEB 1, 2025"

Commit message: updates
Parts:
- removed 3.3V1, HI-V1, VHIGH1: TestPoint, Connector_Pin:Pin_D1.0mm_L10.0mm
- removed C5, C6: 1uF, Capacitor_SMD:C_0805_2012Metric
- removed U2: RP115X, Package_TO_SOT_SMD:SOT-89-5
- added C28: 0.01uF, Capacitor_SMD:C_0805_2012Metric, F.Cu at (53.2, 75.4)
- added C29: 1uF/ 500V, Capacitor_SMD:C_2220_5750Metric, F.Cu at (53.6, 68.6)
- added D16: YELLOW, LED_SMD:LED_0805_2012Metric, F.Cu at (127.4, 85.0)
- added GND1: TestPoint, Connector_Pin:Pin_D1.0mm_L10.0mm, F.Cu at (112.7, 166.9)
- added HIV+1: TestPoint, Connector_Pin:Pin_D1.0mm_L10.0mm, F.Cu at (58.3, 58.1)
- added HIV-1: TestPoint, Connector_Pin:Pin_D1.0mm_L10.0mm, F.Cu at (63.2, 52.4)
- added R36: 4.7k, Resistor_SMD:R_0805_2012Metric, F.Cu at (123.4, 85.1)
- added STG1: TestPoint, Connector_Pin:Pin_D1.0mm_L10.0mm, F.Cu at (63.4, 58.1)
- C2, C3: value 0.1uF -> 10uF
- C27: value 1uF/ 500V -> 150uF/ 450V; footprint Capacitor_SMD:C_2220_5750Metric -> Capacitor_THT:CP_Radial_D18.0mm_P7.50mm
- D4: value GREEN -> YELLOW
- R4: value 715R -> 5M
- U1: value TPS2115APWR -> AP7363-33D-13; footprint TPS2115APWR:PW8 -> AP7363_33D_13:TO252-3L_DIO
- moved R35 86.3 mm to (54.9, 142.8), turned to -90 degrees
- moved C2 32.8 mm to (89.3, 123.7)
- moved C3 28.5 mm to (89.4, 133.7), turned to 0 degrees
- moved U1 28.3 mm to (89.7, 128.5)
- moved R4 22.6 mm to (89.3, 137.6)
- moved C27 18.9 mm to (34.7, 39.1)
- moved D15 14.2 mm to (44.9, 68.6)
- moved D4 9.30 mm to (127.5, 94.3)
- moved R8 9.30 mm to (123.3, 94.3)
- moved DRAIN1 0.89 mm to (60.7, 66.9)
- moved S1 0.14 mm to (134.8, 66.5)
- moved S2 0.14 mm to (128.0, 66.6)
Connections:
- C1 pad 1: GND -> Net-(C1-Pad1)
- C2 pad 1: +VBAT -> VBUS
- C27 pad 1: Net-(D1-A) -> Net-(D15-A)
- C27 pad 2: +500V -> Net-(D1-K)
- C3 pad 1: VBUS -> +3.3V
- D15 pad 2: GND -> Net-(D15-A)
- F1 pad 2: GND -> Net-(D15-A)
- L1 pad 1: VHIGH -> +3.3V
- R1 pad 2: +5V -> VBUS
- R35 pad 2: +5V -> VBUS
- R4 pad 1: GND -> unconnected-(R4-Pad1)
- R4 pad 2: Net-(U1-ILIM) -> +3.3V
- R8 pad 2: +5V -> /BLINK
- T1 pad 6: +500V -> Net-(D1-A)
- T1 pad 7: GND -> Net-(C1-Pad1)
- U1 pad 1: /VSTAT -> VBUS
- U1 pad 3: unconnected-(U1-D1-Pad3) -> +3.3V
- U4 pad 38: unconnected-(U4-IO2-Pad38) -> /BLINK
Routing:
- net +5V: track 159.9 -> 27.2 mm, vias 7 -> 2
- net Net-(D1-A): track 0.00 -> 83.8 mm, vias 0 -> 2
- net +500V: track 80.4 -> 0.00 mm, vias 2 -> 0
- net VHIGH: track 67.1 -> 0.00 mm, vias 3 -> 0
- net +VBAT: track 160.6 -> 101.4 mm, vias 5 -> 4
- net Net-(D15-A): track 0.00 -> 37.2 mm
- net GND: track 403.9 -> 371.5 mm, vias 36 -> 31
- net Net-(JP1-A): track 80.5 -> 86.4 mm
- net +3.3V: track 457.0 -> 462.4 mm, vias 14 -> 13
- net VBUS: track 223.9 -> 228.2 mm
- net Net-(U1-ILIM): track 2.65 -> 0.00 mm
- net Net-(D16-A): track 0.00 -> 2.18 mm
- net /BEEP: track 114.6 -> 112.5 mm
- net Net-(C1-Pad1): track 0.00 -> 1.93 mm, vias 0 -> 1
- net /VSTAT: track 111.0 -> 109.3 mm
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- added copper zone on In2.Cu, net Net-(D1-A)
- removed copper zone on In2.Cu, net +500V
Other:
- board text added: "BLINK"
- board text added: "BOOT"
- board text added: "EN"
- board text added: "HIV+"
- board text added: "HIV-"
- board text added: "STAGE1"

Commit message: PCB v2
Parts:
- removed C27: 150uF/ 450V, Capacitor_THT:CP_Radial_D18.0mm_P7.50mm
- removed STAT1: TestPoint, Connector_Pin:Pin_D1.0mm_L10.0mm
- added C30: 1000pF, Capacitor_SMD:C_0805_2012Metric, F.Cu at (56.6, 98.9)
- added C5: 1000pF, Capacitor_SMD:C_0805_2012Metric, F.Cu at (66.0, 76.2)
- added C6: 0.1uF, Capacitor_SMD:C_0805_2012Metric, F.Cu at (89.8, 108.0)
- added GND2: TestPoint, Connector_Pin:Pin_D1.0mm_L10.0mm, F.Cu at (128.4, 120.2)
- added JP4: SolderJumper_2_Open, Jumper:SolderJumper-2_P1.3mm_Open_RoundedPad1.0x1.5mm, F.Cu at (104.6, 127.8)
- added JP5: SolderJumper_2_Open, Jumper:SolderJumper-2_P1.3mm_Open_RoundedPad1.0x1.5mm, F.Cu at (104.6, 124.7)
- added JP6: SolderJumper_2_Open, Jumper:SolderJumper-2_P1.3mm_Open_RoundedPad1.0x1.5mm, F.Cu at (104.5, 121.7)
- added R37: 100R, Resistor_SMD:R_0805_2012Metric, F.Cu at (63.6, 76.2)
- added R38: 1M, Resistor_SMD:R_1210_3225Metric, F.Cu at (85.9, 104.7)
- added R39: 22k, Resistor_SMD:R_0805_2012Metric, F.Cu at (82.1, 115.6)
- added R40: 10k, Resistor_SMD:R_0805_2012Metric, F.Cu at (82.1, 117.7)
- added R41: 10k, Resistor_SMD:R_0805_2012Metric, F.Cu at (81.6, 104.8)
- added U2: LM393BIPWR, LM393BIPWR:PW0008A-MFG, F.Cu at (86.9, 110.8)
- C28: value 0.01uF -> 100pF
- D10, D11, D12, D5, D6, D7: value ESD9B5.0ST5G -> PESD5V0S1BA; footprint Diode_SMD:D_SOD-923 -> PESD5V0S1BA:SOD323_NXP
- R4: value 5M -> 10k
- moved VBUS1 94.0 mm to (76.1, 90.1)
- moved R4 29.9 mm to (85.0, 108.0), turned to 0 degrees
- moved HIV-1 29.7 mm to (66.9, 81.9)
- moved STG1 26.1 mm to (70.2, 83.3)
- moved HIV+1 25.2 mm to (62.6, 82.9)
- moved R35 2.83 mm to (57.3, 141.3)
- moved U1 2.42 mm to (90.0, 130.9)
- moved C2 2.42 mm to (89.6, 126.1)
- moved D6 2.20 mm to (118.1, 174.0), turned to 180 degrees
- moved D10 1.90 mm to (92.9, 174.9), turned to 180 degrees
- moved C3 1.87 mm to (89.9, 135.5)
- moved D11 1.00 mm to (92.9, 177.3), turned to 180 degrees
- moved D5 1.00 mm to (118.1, 176.3), turned to 180 degrees
- moved R3 0.90 mm to (59.4, 95.1)
- moved D12 0.20 mm to (92.9, 179.6), turned to 180 degrees
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Connections:
- net Net-(D15-A) renamed /Power2/CATHODE
- net Net-(F1-Pad1) renamed /Power2/ANODE
- C28 pad 1: GND -> Net-(Q1-G)
- C28 pad 2: Net-(JP1-A) -> GND
- D10 pad 1: VBUS -> GND
- D10 pad 2: GND -> VBUS
- D11 pad 1: /MCU2/DP_N -> GND
- D11 pad 2: GND -> /MCU2/DP_N
- D12 pad 1: /MCU2/DP_P -> GND
- D12 pad 2: GND -> /MCU2/DP_P
- D5 pad 1: /USB_D+ -> GND
- D5 pad 2: GND -> /USB_D+
- D6 pad 1: /USB_D- -> GND
- D6 pad 2: GND -> /USB_D-
- D7 pad 1: VBUS -> GND
- D7 pad 2: GND -> VBUS
- R24 pad 2: +VBAT -> /BAT_SENSE
- R4 pad 1: unconnected-(R4-Pad1) -> /RAD_IN
- R9 pad 2: +VBAT -> VBUS
- S4 pad 5B: /GPIO15 -> /GPIO16
- S4 pad 6A: +3.3V -> /RAD_IN
- S4 pad 6B: /GPIO16 -> /RAD_IN2
- U4 pad 15: /VSTAT -> unconnected-(U4-IO3-Pad15)
- U4 pad 17: unconnected-(U4-IO9-Pad17) -> /BAT_SENSE
- U4 pad 8: /GPIO15 -> /RAD_IN2
Routing:
- net /VSTAT: track 109.3 -> 0.00 mm, vias 2 -> 0
- net +VBAT: track 101.4 -> 0.00 mm, vias 4 -> 0
- net VBUS: track 228.2 -> 308.5 mm, vias 7 -> 11
- net +5V: track 27.2 -> 106.3 mm, vias 2 -> 3
- net +3.3V: track 462.4 -> 537.0 mm, vias 13 -> 17
- net /RAD_IN: track 0.00 -> 70.4 mm, vias 0 -> 5
- net /BAT_SENSE: track 0.00 -> 56.8 mm, vias 0 -> 3
- net Net-(C1-Pad1): track 1.93 -> 55.0 mm, vias 1 -> 3
- net /BLINK: track 0.00 -> 50.2 mm, vias 0 -> 2
- net GND: track 371.5 -> 421.2 mm, vias 31 -> 40
- net /Power2/CATHODE: track 37.2 -> 78.4 mm
- net Net-(C30-Pad2): track 0.00 -> 41.0 mm, vias 0 -> 2
- net /RAD_IN2: track 0.00 -> 34.1 mm, vias 0 -> 2
- net /GPIO15: track 34.0 -> 0.00 mm, vias 2 -> 0
- net Net-(JP4-A): track 0.00 -> 25.7 mm
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Other:
- board text added: "CS"
- board text added: "DI"
- board text added: "DO"
- board text added: "GND"
- board text added: "SCK"
- board text removed: "HIV+"
- board text removed: "HIV-"
- board text removed: "STAGE1"
