File: Radiation2.kicad_sch (KiCad schematic)
At the start: 0 parts

Commit message: updates
Other:
- sheet MCU2 ports: added BLINK; removed none
- sheet Power2 ports: added BLINK; removed none
- note added: "-change 3.3V regulator chip -add diode arrows -VBAT is missing -sense for radiation hit is missing -add test point names TP5, 8 etc too confusing -order 2.2nF and 1uF/ 500V capacitor -check GPIO46 CIRCUITRY -LED driver --maybe change PWM MOSFET chip TODO: LEAVE ROOM FOR DEV BOARD TO PLUG IN BUILD IN DISPLAY FOR TESTING BATTERY LIFE EYES EVERYWHERE ON THE EGGS"
- note added: "1. Breadboard Delon circuit with input to MCU 2. set PCB up for both with jumpers! 3. design and test input to the ESP32 4. check fuse holder footprint 4. add all of these things to PCB and BOM 5. test SD card functionality 7. check BOM to make sure everything is on it 8. 40 pushups! did 40! SUN FEB 16 9. 40 pushups mon feb 17"
- note removed: "-change 3.3V regulator chip -add LED blink on unused GPIO -add diode arrows -VBAT is missing -sense for radiation hit is missing -fuse clip footprint wrong -add test point names TP5, 8 etc too confusing -add positive and negative for GM tube -order 2.2nF and 1uF/ 500V capacitor -footprint wrong Q2, Q3 -add 10ohm 2W resistor between 5V and pin 2 transformer. gets hot, test higher value resistor -c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"
Changed lines of the file:
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@@
+	(wire
+		(pts
+			(xy 97.79 92.71) (xy 113.03 92.71)
+		)
+		(stroke
+			(width 0)
+			(type default)
+		)
+	)
 	(wire
 		(pts
@@
 	(wire
 		(pts
+			(xy 60.96 38.1) (xy 73.66 38.1)
+		)
+		(stroke
+			(width 0)
+			(type default)
+		)
+	)
+	(wire
+		(pts
 			(xy 60.96 128.27) (xy 73.66 128.27)
 		)
@@
 		)
 	)
-	(text "-change 3.3V regulator chip\n-add LED blink on unused GPIO\n-add diode arrows\n-VBAT is missing\n-sense for radiation hit is missing\n\n-fuse clip footprint wrong \n-add test point names TP5, 8 etc too confusing\n-add positive and negative for GM tube\n-order 2.2nF and 1uF/ 500V capacitor\n-footprint wrong Q2, Q3\n-add 10ohm 2W resistor between 5V and pin 2 transformer. gets hot, test higher value resistor\n-check GPIO46 CIRCUITRY\n-LED driver\n--maybe change PWM MOSFET chip\n\nTODO:\nLEAVE ROOM FOR DEV BOARD TO PLUG IN\nBUILD IN DISPLAY FOR TESTING BATTERY LIFE\nEYES EVERYWHERE ON THE EGGS"
+	(text "1. Breadboard Delon circuit with input to MCU\n2. set PCB up for both with jumpers!\n3. design and test input to the ESP32\n4. check fuse holder footprint\n4. add all of these things to PCB and BOM\n5. test SD card functionality\n7. check BOM to make sure everything is on it\n8. 40 pushups! did 40! SUN FEB 16\n9. 40 pushups mon feb 17"
+		(exclude_from_sim no)
+		(at 177.8 45.72 0)
+		(effects
+			(font
+				(size 1.27 1.27)
+				(thickness 0.254)
+				(bold yes)
+			)
+			(justify left)
+		)
+	)
+	(text "-change 3.3V regulator chip\n-add diode arrows\n-VBAT is missing\n-sense for radiation hit is missing\n-add test point names TP5, 8 etc too confusing\n-order 2.2nF and 1uF/ 500V capacitor\n-check GPIO46 CIRCUITRY\n-LED driver\n--maybe change PWM MOSFET chip\n\nTODO:\nLEAVE ROOM FOR DEV BOARD TO PLUG IN\nBUILD IN DISPLAY FOR TESTING BATTERY LIFE\nEYES EVERYWHERE ON THE EGGS"
 		(exclude_from_sim no)
 		(at 178.054 71.12 0)
@@
 		)
 	)
+	(label "BLINK"
+		(at 62.23 38.1 0)
+		(fields_autoplaced yes)
+		(effects
+			(font
+				(size 1.27 1.27)
+			)
+			(justify left bottom)
+		)
+	)
 	(label "+VBAT"
 		(at 100.33 36.83 0)
@@
 	(label "GPIO38"
 		(at 60.96 120.65 0)
+		(fields_autoplaced yes)
+		(effects
+			(font
+				(size 1.27 1.27)
+			)
+			(justify left bottom)
+		)
+	)
+	(label "BLINK"
+		(at 101.6 92.71 0)
 		(fields_autoplaced yes)
 		(effects
@@
 		(pin "GPIO16" input
 			(at 97.79 90.17 0)
+			(effects
+				(font
+					(size 1.27 1.27)
+				)
+				(justify right)
+			)
+		)
+		(pin "BLINK" input
+			(at 97.79 92.71 0)
 			(effects
 				(font
@@
 			(effects
 				(font
+					(size 1.27 1.27)
+				)
+				(justify left)
+			)
+		)
+		(pin "BLINK" input
+			(at 73.66 38.1 180)
+			(effects
+				(font

Commit message: PCB v2
Other:
- sheet Audio2 ports: added RAD_IN, RAD_IN2; removed GPIO15
- sheet MCU2 ports: added BAT_SENSE, RAD_IN2, VBUS; removed +VBAT, GPIO15, VSTAT
- sheet Power2 ports: added BAT_SENSE, RAD_IN; removed +VBAT, VSTAT
- note added: "-add test point names TP5, 8 etc too confusing -order 2.2nF and 1uF/ 500V capacitor WHILE V2 IS BEING FABBED, TEST: DAC OTG SD CARD TODO: LEAVE ROOM FOR DEV BOARD TO PLUG IN BUILD IN DISPLAY FOR TESTING BATTERY LIFE EYES EVERYWHERE ON THE EGGS LED DRIVER Check GPIO46 CIRCUITRY"
- note added: "NOTES FOR PCB V2 BRINGUP: USE DIP SWITCH FOR RADIATION PULSE"
- note added: "NOTES FROM PCB V1: 3.3V REGULATOR FAILED SHORT BETWEEN VIN AND VOUT"
- note removed: "-change 3.3V regulator chip -add diode arrows -VBAT is missing -sense for radiation hit is missing -add test point names TP5, 8 etc too confusing -order 2.2nF and 1uF/ 500V capacitor -check GPIO46 CIRCUITRY -LED driver --maybe change PWM MOSFET chip TODO: LEAVE ROOM FOR DEV BOARD TO PLUG IN BUILD IN DISPLAY FOR TESTING BATTERY LIFE EYES EVERYWHERE ON THE EGGS"
- note removed: "1. Breadboard Delon circuit with input to MCU 2. set PCB up for both with jumpers! 3. design and test input to the ESP32 4. check fuse holder footprint 4. add all of these things to PCB and BOM 5. test SD card functionality 7. check BOM to make sure everything is on it 8. 40 pushups! did 40! SUN FEB 16 9. 40 pushups mon feb 17"
